Commit message: Update arm_2026 for NEMA17 tuning and teleop control

File: src/arm_2026/description/arm_2026.urdf.xacro (robot description, xacro)
@@ -38,5 +38,5 @@
     <origin xyz="0 0 0.05" rpy="0 0 0"/>
     <axis xyz="0 0 1"/>
-    <limit lower="-3.14" upper="3.14" effort="10" velocity="1.0"/>
+    <limit lower="-3.14" upper="3.14" effort="10" velocity="60.0"/>
   </joint>
   <joint name="shoulder_extension" type="revolute">
